File: hardware/dac.sch (KiCad schematic (older format))
At the start: 7 parts, among them IC4 DAC8562SDGSR, J4 Conn_01x04

Commit message: Last adjustments to hardware before v0.1 release
Parts:
- C13: renamed from C12; LCSC (none) -> C1588; LCSC Part # (none) -> C1588
- C14: renamed from C13; LCSC (none) -> C14663; LCSC Part # (none) -> C14663
- C15: renamed from C14; LCSC (none) -> C14858; LCSC Part # (none) -> C14858
- C16: renamed from C15; LCSC (none) -> C21120; LCSC Part # (none) -> C21120
- R5: LCSC (none) -> C25804; LCSC Part # (none) -> C25804
Changed lines of the file:
@@
 $EndDescr
 $Comp
-L power:GND #PWR033
+L power:GND #PWR039
 U 1 1 5ED3A9D0
 P 6400 3950
-F 0 "#PWR033" H 6400 3700 50  0001 C CNN
+F 0 "#PWR039" H 6400 3700 50  0001 C CNN
 F 1 "GND" V 6405 3822 50  0000 R CNN
 F 2 "" H 6400 3950 50  0001 C CNN
@@
 $EndComp
 $Comp
-L power:GND #PWR034
+L power:GND #PWR040
 U 1 1 5FB5E7F1
 P 6550 2150
-F 0 "#PWR034" H 6550 1900 50  0001 C CNN
+F 0 "#PWR040" H 6550 1900 50  0001 C CNN
 F 1 "GND" H 6555 1977 50  0000 C CNN
 F 2 "" H 6550 2150 50  0001 C CNN
@@
 	6300 3950 6400 3950
 $Comp
-L Device:C C15
+L Device:C C16
 U 1 1 5FB6035A
 P 6550 2000
-F 0 "C15" H 6435 1954 50  0000 R CNN
+F 0 "C16" H 6435 1954 50  0000 R CNN
 F 1 "220n" H 6435 2045 50  0000 R CNN
 F 2 "Capacitor_SMD:C_0603_1608Metric" H 6588 1850 50  0001 C CNN
 F 3 "~" H 6550 2000 50  0001 C CNN
+F 4 "C21120" H 6550 2000 50  0001 C CNN "LCSC Part #"
+F 5 "C21120" H 6550 2000 50  0001 C CNN "LCSC"
 	1    6550 2000
 	1    0    0    -1
 $EndComp
 $Comp
-L Device:C C12
+L Device:C C13
 U 1 1 5FB6078F
 P 4050 2000
-F 0 "C12" H 3935 1954 50  0000 R CNN
+F 0 "C13" H 3935 1954 50  0000 R CNN
 F 1 "1n" H 3935 2045 50  0000 R CNN
 F 2 "Capacitor_SMD:C_0603_1608Metric" H 4088 1850 50  0001 C CNN
 F 3 "~" H 4050 2000 50  0001 C CNN
+F 4 "C1588" H 4050 2000 50  0001 C CNN "LCSC Part #"
+F 5 "C1588" H 4050 2000 50  0001 C CNN "LCSC"
 	1    4050 2000
 	-1   0    0    1
 $EndComp
 $Comp
-L power:GND #PWR031
+L power:GND #PWR037
 U 1 1 5FB62572
 P 4450 2300
-F 0 "#PWR031" H 4450 2050 50  0001 C CNN
+F 0 "#PWR037" H 4450 2050 50  0001 C CNN
 F 1 "GND" H 4455 2127 50  0000 C CNN
 F 2 "" H 4450 2300 50  0001 C CNN
@@
 	4450 2150 4450 2300
 Text GLabel 5150 1850 2    50   Input ~ 0
-dac_avdd
+3v3a
 Text GLabel 4450 4050 0    50   Input ~ 0
-dac_avdd
+3v3a
 Text GLabel 4450 4150 0    50   Input ~ 0
 dac_vref
@@
 Check Layout example in datasheet!!
 $Comp
-L power:+3V3 #PWR032
+L power:+3V3 #PWR038
 U 1 1 5FD27C48
 P 6400 3350
-F 0 "#PWR032" H 6400 3200 50  0001 C CNN
+F 0 "#PWR038" H 6400 3200 50  0001 C CNN
 F 1 "+3V3" H 6415 3523 50  0000 C CNN
 F 2 "" H 6400 3350 50  0001 C CNN
@@
 F 2 "Resistor_SMD:R_0603_1608Metric" V 6330 3550 50  0001 C CNN
 F 3 "~" H 6400 3550 50  0001 C CNN
+F 4 "C25804" H 6400 3550 50  0001 C CNN "LCSC Part #"
+F 5 "C25804" H 6400 3550 50  0001 C CNN "LCSC"
 	1    6400 3550
 	1    0    0    -1
@@
 	6400 3350 6400 3400
 $Comp
-L Device:C C13
+L Device:C C14
 U 1 1 5FB90B4F
 P 4450 2000
-F 0 "C13" H 4565 2046 50  0000 L CNN
+F 0 "C14" H 4565 2046 50  0000 L CNN
 F 1 "100n" H 4565 1955 50  0000 L CNN
 F 2 "Capacitor_SMD:C_0603_1608Metric" H 4488 1850 50  0001 C CNN
 F 3 "~" H 4450 2000 50  0001 C CNN
+F 4 "C14663" H 4450 2000 50  0001 C CNN "LCSC Part #"
+F 5 "C14663" H 4450 2000 50  0001 C CNN "LCSC"
 	1    4450 2000
 	1    0    0    -1
 $EndComp
 $Comp
-L Device:C C14
+L Device:C C15
 U 1 1 5FE5ED0F
 P 4900 2000
-F 0 "C14" H 5015 2046 50  0000 L CNN
+F 0 "C15" H 5015 2046 50  0000 L CNN
 F 1 "100p" H 5015 1955 50  0000 L CNN
 F 2 "Capacitor_SMD:C_0603_1608Metric" H 4938 1850 50  0001 C CNN
 F 3 "~" H 4900 2000 50  0001 C CNN
+F 4 "C14858" H 4900 2000 50  0001 C CNN "LCSC Part #"
+F 5 "C14858" H 4900 2000 50  0001 C CNN "LCSC"
 	1    4900 2000
 	1    0    0    -1
@@
 AR Path="/5FECC484" Ref="#PWR?"  Part="1"
 AR Path="/5FDE753F/5FECC484" Ref="#PWR?"  Part="1"
-AR Path="/5ED37B53/5FECC484" Ref="#PWR030"  Part="1"
-F 0 "#PWR030" H 3700 1700 50  0001 C CNN
+AR Path="/5ED37B53/5FECC484" Ref="#PWR036"  Part="1"
+F 0 "#PWR036" H 3700 1700 50  0001 C CNN
 F 1 "+3.3VA" V 3715 1977 50  0000 L CNN
 F 2 "" H 3700 1850 50  0001 C CNN
