File: hardware/encoder.sch (KiCad schematic (older format))
At the start: 3 parts

Commit message: Minor adjustments to schematics before PCB
Parts:
- R27, R28: renamed from R?; footprint (none) -> Resistor_SMD:R_0603_1608Metric
- VR11: renamed from VR?; footprint PEC11R4220FS0024 -> PEC11R-4220F-S0024:PEC11R4220FS0024
Changed lines of the file:
@@
 $Descr A4 11693 8268
 encoding utf-8
-Sheet 10 10
+Sheet 9 11
 Title ""
 Date ""
@@
 $EndDescr
 $Comp
-L PEC11R-4220F-S0024:PEC11R-4220F-S0024 VR?
+L PEC11R-4220F-S0024:PEC11R-4220F-S0024 VR11
 U 1 1 5FDF0E4F
 P 5950 3050
-F 0 "VR?" H 6800 3500 50  0000 L CNN
+F 0 "VR11" H 6800 3500 50  0000 L CNN
 F 1 "PEC11R-4220F-S0024" H 6800 3400 50  0000 L CNN
-F 2 "PEC11R4220FS0024" H 6800 3350 50  0001 L CNN
+F 2 "PEC11R-4220F-S0024:PEC11R4220FS0024" H 6800 3350 50  0001 L CNN
 F 3 "https://www.bourns.com/docs/Product-Datasheets/PEC11R.pdf" H 6800 3250 50  0001 L CNN
 F 4 "Bourns 24 Pulse Incremental Mechanical Rotary Encoder with a 6 mm Flat Shaft (Not Indexed), Through Hole" H 6800 3150 50  0001 L CNN "Description"
@@
 $EndComp
 $Comp
-L power:GND #PWR?
+L power:GND #PWR0101
 U 1 1 5FDF2434
 P 4950 3050
-F 0 "#PWR?" H 4950 2800 50  0001 C CNN
+F 0 "#PWR0101" H 4950 2800 50  0001 C CNN
 F 1 "GND" V 4955 2922 50  0000 R CNN
 F 2 "" H 4950 3050 50  0001 C CNN
@@
 	1    4950 3050
 	0    1    1    0
-$EndComp
-$Comp
-L power:GND #PWR?
-U 1 1 5FDF296D
-P 5950 3050
-F 0 "#PWR?" H 5950 2800 50  0001 C CNN
-F 1 "GND" V 5955 2922 50  0000 R CNN
-F 2 "" H 5950 3050 50  0001 C CNN
-F 3 "" H 5950 3050 50  0001 C CNN
-	1    5950 3050
-	0    -1   -1   0
-$EndComp
-$Comp
-L power:GND #PWR?
-U 1 1 5FDF36EB
-P 5450 2200
-F 0 "#PWR?" H 5450 1950 50  0001 C CNN
-F 1 "GND" H 5455 2027 50  0000 C CNN
-F 2 "" H 5450 2200 50  0001 C CNN
-F 3 "" H 5450 2200 50  0001 C CNN
-	1    5450 2200
-	-1   0    0    1
-$EndComp
-$Comp
-L power:GND #PWR?
-U 1 1 5FDF3F6F
-P 5450 3550
-F 0 "#PWR?" H 5450 3300 50  0001 C CNN
-F 1 "GND" H 5455 3377 50  0000 C CNN
-F 2 "" H 5450 3550 50  0001 C CNN
-F 3 "" H 5450 3550 50  0001 C CNN
-	1    5450 3550
-	1    0    0    -1
 $EndComp
 Wire Wire Line
@@
 P 5450 1750
 AR Path="/5ED37B53/5FDF7D49" Ref="#PWR?"  Part="1"
-AR Path="/5FDF0A57/5FDF7D49" Ref="#PWR?"  Part="1"
-F 0 "#PWR?" H 5450 1600 50  0001 C CNN
+AR Path="/5FDF0A57/5FDF7D49" Ref="#PWR0102"  Part="1"
+F 0 "#PWR0102" H 5450 1600 50  0001 C CNN
 F 1 "+3V3" H 5465 1923 50  0000 C CNN
 F 2 "" H 5450 1750 50  0001 C CNN
@@
 P 5150 2100
 AR Path="/5ED37B53/5FDF7D4F" Ref="R?"  Part="1"
-AR Path="/5FDF0A57/5FDF7D4F" Ref="R?"  Part="1"
-F 0 "R?" H 5220 2146 50  0000 L CNN
+AR Path="/5FDF0A57/5FDF7D4F" Ref="R27"  Part="1"
+F 0 "R27" H 5220 2146 50  0000 L CNN
 F 1 "10k" H 5220 2055 50  0000 L CNN
-F 2 "" V 5080 2100 50  0001 C CNN
+F 2 "Resistor_SMD:R_0603_1608Metric" V 5080 2100 50  0001 C CNN
 F 3 "~" H 5150 2100 50  0001 C CNN
 	1    5150 2100
@@
 P 5750 2100
 AR Path="/5ED37B53/5FDFB593" Ref="R?"  Part="1"
-AR Path="/5FDF0A57/5FDFB593" Ref="R?"  Part="1"
-F 0 "R?" H 5820 2146 50  0000 L CNN
+AR Path="/5FDF0A57/5FDFB593" Ref="R28"  Part="1"
+F 0 "R28" H 5820 2146 50  0000 L CNN
 F 1 "10k" H 5820 2055 50  0000 L CNN
-F 2 "" V 5680 2100 50  0001 C CNN
+F 2 "Resistor_SMD:R_0603_1608Metric" V 5680 2100 50  0001 C CNN
 F 3 "~" H 5750 2100 50  0001 C CNN
 	1    5750 2100
@@
 	5750 1800 5750 1950
 Connection ~ 5450 1800
+$Comp
+L power:GND #PWR0103
+U 1 1 5FF3D410
+P 5450 2200
+F 0 "#PWR0103" H 5450 1950 50  0001 C CNN
+F 1 "GND" H 5455 2027 50  0000 C CNN
+F 2 "" H 5450 2200 50  0001 C CNN
+F 3 "" H 5450 2200 50  0001 C CNN
+	1    5450 2200
+	-1   0    0    1
+$EndComp
+$Comp
+L power:GND #PWR0104
+U 1 1 5FF3E986
+P 5450 3550
+F 0 "#PWR0104" H 5450 3300 50  0001 C CNN
+F 1 "GND" H 5455 3377 50  0000 C CNN
+F 2 "" H 5450 3550 50  0001 C CNN
+F 3 "" H 5450 3550 50  0001 C CNN
+	1    5450 3550
+	1    0    0    -1
+$EndComp
+$Comp
+L power:GND #PWR0105
+U 1 1 5FF3FBE0
+P 5950 3050
+F 0 "#PWR0105" H 5950 2800 50  0001 C CNN
+F 1 "GND" H 5955 2877 50  0000 C CNN
+F 2 "" H 5950 3050 50  0001 C CNN
+F 3 "" H 5950 3050 50  0001 C CNN
+	1    5950 3050
+	0    -1   -1   0
+$EndComp
 $EndSCHEMATC

Commit message: Last adjustments to hardware before v0.1 release
Parts:
- R27, R28: LCSC (none) -> C25804; LCSC Part # (none) -> C25804
Changed lines of the file:
@@
 $EndComp
 $Comp
-L power:GND #PWR0101
+L power:GND #PWR0108
 U 1 1 5FDF2434
 P 4950 3050
-F 0 "#PWR0101" H 4950 2800 50  0001 C CNN
+F 0 "#PWR0108" H 4950 2800 50  0001 C CNN
 F 1 "GND" V 4955 2922 50  0000 R CNN
 F 2 "" H 4950 3050 50  0001 C CNN
@@
 P 5450 1750
 AR Path="/5ED37B53/5FDF7D49" Ref="#PWR?"  Part="1"
-AR Path="/5FDF0A57/5FDF7D49" Ref="#PWR0102"  Part="1"
-F 0 "#PWR0102" H 5450 1600 50  0001 C CNN
+AR Path="/5FDF0A57/5FDF7D49" Ref="#PWR0109"  Part="1"
+F 0 "#PWR0109" H 5450 1600 50  0001 C CNN
 F 1 "+3V3" H 5465 1923 50  0000 C CNN
 F 2 "" H 5450 1750 50  0001 C CNN
@@
 F 2 "Resistor_SMD:R_0603_1608Metric" V 5080 2100 50  0001 C CNN
 F 3 "~" H 5150 2100 50  0001 C CNN
+F 4 "C25804" H 5150 2100 50  0001 C CNN "LCSC Part #"
+F 5 "C25804" H 5150 2100 50  0001 C CNN "LCSC"
 	1    5150 2100
 	1    0    0    -1
@@
 F 2 "Resistor_SMD:R_0603_1608Metric" V 5680 2100 50  0001 C CNN
 F 3 "~" H 5750 2100 50  0001 C CNN
+F 4 "C25804" H 5750 2100 50  0001 C CNN "LCSC Part #"
+F 5 "C25804" H 5750 2100 50  0001 C CNN "LCSC"
 	1    5750 2100
 	1    0    0    -1
@@
 Connection ~ 5450 1800
 $Comp
-L power:GND #PWR0103
+L power:GND #PWR0110
 U 1 1 5FF3D410
 P 5450 2200
-F 0 "#PWR0103" H 5450 1950 50  0001 C CNN
+F 0 "#PWR0110" H 5450 1950 50  0001 C CNN
 F 1 "GND" H 5455 2027 50  0000 C CNN
 F 2 "" H 5450 2200 50  0001 C CNN
@@
 $EndComp
 $Comp
-L power:GND #PWR0104
+L power:GND #PWR0111
 U 1 1 5FF3E986
 P 5450 3550
-F 0 "#PWR0104" H 5450 3300 50  0001 C CNN
+F 0 "#PWR0111" H 5450 3300 50  0001 C CNN
 F 1 "GND" H 5455 3377 50  0000 C CNN
 F 2 "" H 5450 3550 50  0001 C CNN
@@
 $EndComp
 $Comp
-L power:GND #PWR0105
+L power:GND #PWR0112
 U 1 1 5FF3FBE0
 P 5950 3050
-F 0 "#PWR0105" H 5950 2800 50  0001 C CNN
+F 0 "#PWR0112" H 5950 2800 50  0001 C CNN
 F 1 "GND" H 5955 2877 50  0000 C CNN
 F 2 "" H 5950 3050 50  0001 C CNN
