File: hardware/faders_pots.sch (KiCad schematic (older format))
At the start: 18 parts

Commit message: Minor adjustments to schematics before PCB
Parts:
- removed RV?: Alpha B10k, symbol Device:R_POT
- added C20, C21, C22, C23, C24, C25, C26, C27, C28, C29: 100n, Capacitor_SMD:C_0603_1608Metric, symbol Device:C
- added VR10: Alpha B10k, Potentiometer_THT:Potentiometer_Alpha_RD901F-40-00D_Single_Vertical, symbol Device:R_POT
- R18, R19, R20, R21, R22, R23, R24, R25: renamed from R?; footprint (none) -> Resistor_SMD:R_0603_1608Metric
- VR1, VR2, VR3, VR4, VR5, VR6, VR7, VR8: renamed from VR?; footprint PTL3010R1103B2 -> PTL30-10R1-103B2:PTL3010R1103B2
- VR9: renamed from RV?; footprint (none) -> Potentiometer_THT:Potentiometer_Alpha_RD901F-40-00D_Single_Vertical
Connections:
- net +3V3: no longer VR1.1 (CCW), VR2.1 (CCW), VR3.1 (CCW), VR4.1 (CCW), VR5.1 (CCW), VR6.1 (CCW), VR7.1 (CCW), VR8.1 (CCW), VR9.3
- net GND: now also C20.1, C21.1, C22.1, C23.1, C24.1, C25.1, C26.1, C27.1, C28.1, C29.1, VR10.1
- net fader_a: now also C20.2
- net fader_b: now also C22.2
- net fader_c: now also C24.2
- net fader_d: now also C26.2
- net fader_e: now also C21.2
- net fader_f: now also C23.2
- net fader_g: now also C25.2
- net fader_h: now also C27.2
- net pot_a: now also C28.2
- net pot_b: now also C29.2, VR10.2
- new net +3.3VA: VR1.1 (CCW), VR10.3, VR2.1 (CCW), VR3.1 (CCW), VR4.1 (CCW), VR5.1 (CCW), VR6.1 (CCW), VR7.1 (CCW), VR8.1 (CCW), VR9.3
Other:
- moved on the sheet: VR9

Commit message: Last adjustments to hardware before v0.1 release
Parts:
- C21: renamed from C20; LCSC (none) -> C14663; LCSC Part # (none) -> C14663
- C22: renamed from C21; LCSC (none) -> C14663; LCSC Part # (none) -> C14663
- C23: renamed from C22; LCSC (none) -> C14663; LCSC Part # (none) -> C14663
- C24: renamed from C23; LCSC (none) -> C14663; LCSC Part # (none) -> C14663
- C25: renamed from C24; LCSC (none) -> C14663; LCSC Part # (none) -> C14663
- C26: renamed from C25; LCSC (none) -> C14663; LCSC Part # (none) -> C14663
- C27: renamed from C26; LCSC (none) -> C14663; LCSC Part # (none) -> C14663
- C28: renamed from C27; LCSC (none) -> C14663; LCSC Part # (none) -> C14663
- C29: renamed from C28; LCSC (none) -> C14663; LCSC Part # (none) -> C14663
- C30: renamed from C29; LCSC (none) -> C14663; LCSC Part # (none) -> C14663
- R18, R19, R20, R21, R22, R23, R24, R25: LCSC (none) -> C22962; LCSC Part # (none) -> C22962
- renumbered VR5 to VR2, VR2 to VR3, VR6 to VR4, VR3 to VR5, VR7 to VR6, VR4 to VR7
