File: hardware/frank_counts.kicad_pcb (KiCad board)
At the start: 2 copper layers, 100 x 100 mm, 137 parts, among them IC1 SN74AHCT1G125DBVR, IC2 SN74AHCT1G125DBVR, IC3 TLC59482DBQ, IC4 DAC8562SDGSR, IC5 ADP150AUJZ-3.3-R7, J1 PJ398SM, J10 PJ398SM, J11 Conn_02x05_Odd_Even, J12 Conn_01x03, J13 Conn_01x01, J2 PJ398SM, J3 Conn_01x04, J4 Conn_01x04, J5 PJ398SM, J6 PJ398SM, J7 PJ398SM, J8 Eurorack PWR, J9 PJ398SM, Q1 MMBT3904, U1 STM32L452RETx, U2 TL072, U3 LM1117-3.3, U4 R-78E5.0-0.5, U5 LM4040DBZ-10, U6 MCP6002-xMS, Y1 ABM3-8.000MHZ

Commit message: Last adjustments to hardware before v0.1 release
Parts:
- added C39: 1u, Capacitor_SMD:C_0603_1608Metric, B.Cu at (95.3, 105.5)
- added D1: BAT54S, Package_TO_SOT_SMD:SOT-23, B.Cu at (130.0, 99.0)
- added R39: 10k, Resistor_SMD:R_0603_1608Metric, B.Cu at (92.0, 62.5)
- C19: renamed from C18; value 7p -> 10p
- C2, C4: value 22p -> 22-26p
- C20: renamed from C19; value 7p -> 10p
- R1: value 768R -> 750R
- R12, R13: value 500 -> 470R
- moved C15 3.41 mm to (108.9, 78.6)
- moved C14 3.27 mm to (108.9, 75.2)
- moved C41 3.19 mm to (101.9, 105.7)
- moved U5 3.17 mm to (99.1, 105.8)
- moved C13 0.05 mm to (108.9, 76.9)
- renumbered C44 to C12, C12 to C13, C13 to C14, C14 to C15, C15 to C16, C16 to C17, C17 to C18, C20 to C21, C21 to C22, C22 to C23, C23 to C24, C24 to C25, C25 to C26, C26 to C27, C27 to C28, C28 to C29, C29 to C30, C30 to C31, C31 to C32, C32 to C33, C33 to C34, C34 to C35, C35 to C36, C36 to C37, C37 to C38, C38 to C40, C39 to C41, C40 to C42, C41 to C43, C42 to C44, C43 to C45, D9 to D10, D10 to D11, D11 to D12, D12 to D13, D13 to D14, D8 to D2, D7 to D3, D6 to D4, D1 to D6, D2 to D7, D3 to D8, D4 to D9, VR5 to VR2, VR2 to VR3, VR6 to VR4, VR3 to VR5, VR7 to VR6, VR4 to VR7
Connections:
- net dac_avdd renamed 3v3a
- net jtag_nrst renamed jtag_reset
Routing:
- net GND: track 76.0 -> 89.3 mm, vias 109 -> 244
- net +3V3: track 375.0 -> 387.0 mm
- net jack_detect: track 74.1 -> 78.0 mm, vias 3 -> 4
- net Net-(R39-Pad1): track 0.00 -> 2.82 mm
- net VEE: track 21.3 -> 23.8 mm
- net dac_vref: track 84.6 -> 82.4 mm
- net ref_-10v: track 106.2 -> 104.8 mm
- net encoder_sw: vias 2 -> 1
