File: hardware/frank_counts.sch (KiCad schematic (older format))
At the start: 1 part

Commit message: Minor adjustments to schematics before PCB
Parts:
- added C1: 4u7, Capacitor_SMD:C_0603_1608Metric, symbol Device:C
- added C2, C4: 22p, Capacitor_SMD:C_0603_1608Metric, symbol Device:C
- added C3, C5, C6, C7, C9: 100n, Capacitor_SMD:C_0603_1608Metric, symbol Device:C
- added C8: 1u, Capacitor_SMD:C_0603_1608Metric, symbol Device:C
- added H1, H2: MountingHole_Pad, MountingHole:MountingHole_3.2mm_M3, symbol Mechanical:MountingHole_Pad
- added R1: 768R, Resistor_SMD:R_0603_1608Metric, symbol Device:R
- added Y1: ABM3-8.000MHZ, Crystal:Crystal_SMD_Abracon_ABM3-2Pin_5.0x3.2mm_HandSoldering, symbol Device:Crystal
- gave numbers to parts that had none: 1
Connections:
- net led_gsclk: now also U1.35 (PB14); no longer U1.41 (PA8)
- net +3V3: now reaches U1.1 (VBAT)
- net +3V3: now also U1.19 (VDD), U1.32 (VDD), U1.64 (VDD), C1.1, C3.1, C5.1, C6.1, C7.1
- net GND: now reaches U1.12 (VSSA)
- net GND: now also U1.18 (VSS), U1.31 (VSS), U1.47 (VSS), U1.63 (VSS), C1.2, C2.1, C3.2, C4.1, C5.2, C6.2, C7.2, C8.2, C9.2, H1.1, H2.1
- net +3.3VA: now reaches U1.13 (VDDA)
- net +3.3VA: now also C8.1, C9.1
- net jtag_rst renamed debug_trst
- net osc_in renamed hse_in
- net hse_in: now also C2.2, Y1.2
- net osc_out renamed hse_out
- net hse_out: now also R1.2
- new net: C4.2, R1.1, Y1.1
- no-connect marks 0 -> 10
Other:
- note added: "Bypass caps"
- note added: "Crystal oscillator"
- note added: "v_ee, v_cc, 5v, 3v3, 3.3va, ref_-10v"
- note removed: "TODO:\nJTAG connector\nOscillator\nUSART connector (header)\nSome test headers?"
- moved on the sheet: U1

Commit message: Last adjustments to hardware before v0.1 release
Parts:
- added D1: BAT54S, Package_TO_SOT_SMD:SOT-23, symbol Diode:BAT54S
- added R39: 10k, Resistor_SMD:R_0603_1608Metric, symbol Device:R
- C1: LCSC (none) -> C19666; LCSC Part # (none) -> C19666
- C2, C4: value 22p -> 22-26p; LCSC (none) -> C388039; LCSC Part # (none) -> C388039
- C3, C5, C6, C7, C9: LCSC (none) -> C14663; LCSC Part # (none) -> C14663
- C8: LCSC (none) -> C15849; LCSC Part # (none) -> C15849
- R1: value 768R -> 750R; LCSC (none) -> C23241; LCSC Part # (none) -> C23241
Connections:
- net +3V3: now also D1.2
- net GND: now also D1.1, R39.2
- net jack_detect: now also D1.3
- net at U1.60 (PH3): now also R39.1
- net jtag_nrst renamed jtag_reset
- no-connect marks 10 -> 9
Other:
- note added: "BOOT0 needs to\nbe tied to GND"
- moved on the sheet: U1
