File: hardware/power_ref.sch (KiCad schematic (older format))
At the start: 22 parts, among them IC5 ADP150AUJZ-3.3-R7, J8 Eurorack PWR, U3 LM1117-3.3, U4 R-78E5.0-0.5, U5 LM4040DBZ-10

Commit message: Last adjustments to hardware before v0.1 release
Parts:
- added C39: 1u, Capacitor_SMD:C_0603_1608Metric, symbol Device:C
- C31: renamed from C30; LCSC (none) -> C15850; LCSC Part # (none) -> C15850
- C32: renamed from C31; LCSC (none) -> C15850; LCSC Part # (none) -> C15850
- C33: renamed from C32; LCSC (none) -> C14663; LCSC Part # (none) -> C14663
- C34: renamed from C33; LCSC (none) -> C15850; LCSC Part # (none) -> C15850
- C35: renamed from C34; LCSC (none) -> C14663; LCSC Part # (none) -> C14663
- C36: renamed from C35; LCSC (none) -> C45783; LCSC Part # (none) -> C45783
- C37: renamed from C36; LCSC (none) -> C45783; LCSC Part # (none) -> C45783
- C38: renamed from C37; LCSC (none) -> C45783; LCSC Part # (none) -> C45783
- C40: renamed from C38; LCSC (none) -> C15849; LCSC Part # (none) -> C15849
- C41: renamed from C39; LCSC (none) -> C15849; LCSC Part # (none) -> C15849
- C42: renamed from C40; LCSC (none) -> C15849; LCSC Part # (none) -> C15849
- D11: renamed from D10; LCSC (none) -> C8598; LCSC Part # (none) -> C8598
- D12: renamed from D11; LCSC (none) -> C8598; LCSC Part # (none) -> C8598
- FB1, FB2: LCSC (none) -> C1015; LCSC Part # (none) -> C1015
- L1: LCSC (none) -> C1035; LCSC Part # (none) -> C1035
- R26: LCSC (none) -> C4177; LCSC Part # (none) -> C4177
- U3: LCSC (none) -> C6186; LCSC Part # (none) -> C6186
Connections:
- net GND: now also C39.2
- net VEE: now also C39.1
Other:
- note added: "consumption ca. 250mA max (witth all LEDs on 100% brightness)"
- note removed: "out ca. 250mA max (witth all LEDs on 100% brightness)"
