File: hardware/trigger_input.sch (KiCad schematic (older format))
At the start: 7 parts, among them J7 PJ398SM, Q1 MMBT3904

Commit message: Last adjustments to hardware before v0.1 release
Parts:
- Q1: LCSC (none) -> C20526; LCSC Part # (none) -> C20526
- R14, R15: LCSC (none) -> C25803; LCSC Part # (none) -> C25803
- R16: LCSC (none) -> C4216; LCSC Part # (none) -> C4216
- R17: LCSC (none) -> C25804; LCSC Part # (none) -> C25804
- renumbered D9 to D10
Changed lines of the file:
@@
 F 2 "Package_TO_SOT_SMD:SOT-23" H 7100 3225 50  0001 L CIN
 F 3 "https://www.fairchildsemi.com/datasheets/2N/2N3904.pdf" H 6900 3300 50  0001 L CNN
+F 4 "C20526" H 6900 3300 50  0001 C CNN "LCSC Part #"
+F 5 "C20526" H 6900 3300 50  0001 C CNN "LCSC"
 	1    6900 3300
 	1    0    0    -1
@@
 F 2 "Resistor_SMD:R_0603_1608Metric" V 6930 2750 50  0001 C CNN
 F 3 "~" H 7000 2750 50  0001 C CNN
+F 4 "C25804" H 7000 2750 50  0001 C CNN "LCSC Part #"
+F 5 "C25804" H 7000 2750 50  0001 C CNN "LCSC"
 	1    7000 2750
 	1    0    0    -1
@@
 F 2 "Resistor_SMD:R_0603_1608Metric" V 4430 3850 50  0001 C CNN
 F 3 "~" H 4500 3850 50  0001 C CNN
+F 4 "C25803" H 4500 3850 50  0001 C CNN "LCSC Part #"
+F 5 "C25803" H 4500 3850 50  0001 C CNN "LCSC"
 	1    4500 3850
 	1    0    0    -1
@@
 F 2 "Resistor_SMD:R_0603_1608Metric" V 5430 3300 50  0001 C CNN
 F 3 "~" H 5500 3300 50  0001 C CNN
+F 4 "C25803" H 5500 3300 50  0001 C CNN "LCSC Part #"
+F 5 "C25803" H 5500 3300 50  0001 C CNN "LCSC"
 	1    5500 3300
 	0    1    1    0
@@
 F 2 "Resistor_SMD:R_0603_1608Metric" V 6280 3850 50  0001 C CNN
 F 3 "~" H 6350 3850 50  0001 C CNN
+F 4 "C4216" H 6350 3850 50  0001 C CNN "LCSC Part #"
+F 5 "C4216" H 6350 3850 50  0001 C CNN "LCSC"
 	1    6350 3850
 	1    0    0    -1
@@
 	4500 4000 4500 4150
 $Comp
-L power:+3.3V #PWR046
+L power:+3.3V #PWR052
 U 1 1 5ED6C9CF
 P 7000 2500
-F 0 "#PWR046" H 7000 2350 50  0001 C CNN
+F 0 "#PWR052" H 7000 2350 50  0001 C CNN
 F 1 "+3.3V" H 7015 2673 50  0000 C CNN
 F 2 "" H 7000 2500 50  0001 C CNN
@@
 Connection ~ 6350 3300
 $Comp
-L power:GND #PWR045
+L power:GND #PWR051
 U 1 1 5ED7253E
 P 6350 4150
-F 0 "#PWR045" H 6350 3900 50  0001 C CNN
+F 0 "#PWR051" H 6350 3900 50  0001 C CNN
 F 1 "GND" H 6355 3977 50  0000 C CNN
 F 2 "" H 6350 4150 50  0001 C CNN
@@
 	6350 4150 6350 4000
 $Comp
-L power:GND #PWR047
+L power:GND #PWR053
 U 1 1 5ED73092
 P 7000 4150
-F 0 "#PWR047" H 7000 3900 50  0001 C CNN
+F 0 "#PWR053" H 7000 3900 50  0001 C CNN
 F 1 "GND" H 7005 3977 50  0000 C CNN
 F 2 "" H 7000 4150 50  0001 C CNN
@@
 	4100 3400 4500 3400
 $Comp
-L power:GND #PWR043
+L power:GND #PWR049
 U 1 1 5ED63404
 P 4450 3000
-F 0 "#PWR043" H 4450 2750 50  0001 C CNN
+F 0 "#PWR049" H 4450 2750 50  0001 C CNN
 F 1 "GND" H 4455 2827 50  0000 C CNN
 F 2 "" H 4450 3000 50  0001 C CNN
@@
 P 5000 3750
 AR Path="/5FCA3E21/5FDB7947" Ref="D?"  Part="1"
-AR Path="/5ED4085B/5FDB7947" Ref="D9"  Part="1"
-F 0 "D9" V 4954 3830 50  0000 L CNN
+AR Path="/5ED4085B/5FDB7947" Ref="D10"  Part="1"
+F 0 "D10" V 4954 3830 50  0000 L CNN
 F 1 "B72500D0160H060" V 5045 3830 50  0000 L CNN
 F 2 "Diode_SMD:D_0603_1608Metric" H 5000 3750 50  0001 C CNN
@@
 AR Path="/5ED37B53/5FB5AC07/5FDB794E" Ref="#PWR?"  Part="1"
 AR Path="/5FCA3E21/5FDB794E" Ref="#PWR?"  Part="1"
-AR Path="/5ED4085B/5FDB794E" Ref="#PWR044"  Part="1"
-F 0 "#PWR044" H 5000 3900 50  0001 C CNN
+AR Path="/5ED4085B/5FDB794E" Ref="#PWR050"  Part="1"
+F 0 "#PWR050" H 5000 3900 50  0001 C CNN
 F 1 "GND" V 5005 4022 50  0000 R CNN
 F 2 "" H 5000 4150 50  0001 C CNN
