File: hardware/trigger_output.sch (KiCad schematic (older format))
At the start: 8 parts

Commit message: Minor adjustments to schematics before PCB
Parts:
- removed J?: TRIGGER_OUT_A, symbol thonkiconn_jackSocket_fuzzySi:fuzzySI_thonkiconn
- removed J?: TRIGGER_OUT_B, symbol thonkiconn_jackSocket_fuzzySi:fuzzySI_thonkiconn
- added J1, J2: PJ398SM, Connector_Audio:Jack_3.5mm_QingPu_WQP-PJ398SM_Vertical_CircularHoles, symbol Connector:AudioJack2_SwitchT
- C10, C11: renamed from C?; footprint (none) -> Capacitor_SMD:C_0603_1608Metric
- IC1, IC2: renamed from IC?; footprint SOT95P280X145-5N -> SN74AHCT1G125DBVR:SOT95P280X145-5N
- R2, R3: renamed from R?; footprint (none) -> Resistor_SMD:R_0603_1608Metric
Connections:
- net GND: now also J1.S, J1.TN, J2.S, J2.TN
- net at R2.1: now also J1.T
- net at R3.1: now also J2.T
Changed lines of the file:
@@
 $Descr A4 11693 8268
 encoding utf-8
-Sheet 9 10
+Sheet 2 11
 Title ""
 Date ""
@@
 Text HLabel 3850 3900 0    50   Input ~ 0
 trigger_out_b
-$Comp
-L thonkiconn_jackSocket_fuzzySi:fuzzySI_thonkiconn J?
-U 1 1 5FDC2D9B
-P 6450 2550
-AR Path="/5ED37B53/5FB5AC07/5FDC2D9B" Ref="J?"  Part="1"
-AR Path="/5FDBBE2F/5FDC2D9B" Ref="J?"  Part="1"
-F 0 "J?" H 6162 2526 50  0000 R CNN
-F 1 "TRIGGER_OUT_A" H 6162 2617 50  0000 R CNN
-F 2 "" H 6700 2650 50  0001 C CNN
-F 3 "" H 6700 2650 50  0001 C CNN
-	1    6450 2550
-	-1   0    0    1
-$EndComp
-$Comp
-L power:GND #PWR?
-U 1 1 5FDC2DA1
-P 6650 2350
-AR Path="/5ED37B53/5FB5AC07/5FDC2DA1" Ref="#PWR?"  Part="1"
-AR Path="/5FDBBE2F/5FDC2DA1" Ref="#PWR0167"  Part="1"
-F 0 "#PWR0167" H 6650 2100 50  0001 C CNN
-F 1 "GND" V 6655 2222 50  0000 R CNN
-F 2 "" H 6650 2350 50  0001 C CNN
-F 3 "" H 6650 2350 50  0001 C CNN
-	1    6650 2350
-	-1   0    0    1
-$EndComp
-Wire Wire Line
-	6650 2350 6650 2400
-Wire Wire Line
-	6250 2550 6250 2400
-Wire Wire Line
-	6250 2400 6650 2400
-Connection ~ 6650 2400
-Wire Wire Line
-	6650 2400 6650 2450
 Wire Wire Line
 	5200 2650 5650 2650
@@
 P 4200 2650
 AR Path="/5ED37B53/5FB5AC07/5FDC3D71" Ref="#PWR?"  Part="1"
-AR Path="/5FDBBE2F/5FDC3D71" Ref="#PWR0168"  Part="1"
-F 0 "#PWR0168" H 4200 2400 50  0001 C CNN
+AR Path="/5FDBBE2F/5FDC3D71" Ref="#PWR011"  Part="1"
+F 0 "#PWR011" H 4200 2400 50  0001 C CNN
 F 1 "GND" V 4205 2522 50  0000 R CNN
 F 2 "" H 4200 2650 50  0001 C CNN
@@
 $EndComp
 $Comp
-L SN74AHCT1G125DBVR:SN74AHCT1G125DBVR IC?
+L SN74AHCT1G125DBVR:SN74AHCT1G125DBVR IC1
 U 1 1 5FDC47DC
 P 4200 2650
-F 0 "IC?" H 4700 2915 50  0000 C CNN
+F 0 "IC1" H 4700 2915 50  0000 C CNN
 F 1 "SN74AHCT1G125DBVR" H 4700 2824 50  0000 C CNN
-F 2 "SOT95P280X145-5N" H 5050 2750 50  0001 L CNN
+F 2 "SN74AHCT1G125DBVR:SOT95P280X145-5N" H 5050 2750 50  0001 L CNN
 F 3 "http://www.ti.com/lit/ds/symlink/sn74ahct1g125.pdf" H 5050 2650 50  0001 L CNN
 F 4 "74AHCT Single Tri-state Bus Buffer SOT23 SN74AHCT1G125DBVR, Bus Buffer, HCT, 8.5 ns@ 50 pF, 8mA 4.5 ??? 5.5 V 5-Pin SOT-23" H 5050 2550 50  0001 L CNN "Description"
@@
 P 4200 2850
 AR Path="/5ED37B53/5FB5AC07/5FDC7341" Ref="#PWR?"  Part="1"
-AR Path="/5FDBBE2F/5FDC7341" Ref="#PWR0169"  Part="1"
-F 0 "#PWR0169" H 4200 2600 50  0001 C CNN
+AR Path="/5FDBBE2F/5FDC7341" Ref="#PWR012"  Part="1"
+F 0 "#PWR012" H 4200 2600 50  0001 C CNN
 F 1 "GND" V 4205 2722 50  0000 R CNN
 F 2 "" H 4200 2850 50  0001 C CNN
@@
 P 5200 2750
 AR Path="/5FDF6408/5FDC8A1E" Ref="#PWR?"  Part="1"
-AR Path="/5FDBBE2F/5FDC8A1E" Ref="#PWR0170"  Part="1"
-F 0 "#PWR0170" H 5200 2600 50  0001 C CNN
+AR Path="/5FDBBE2F/5FDC8A1E" Ref="#PWR015"  Part="1"
+F 0 "#PWR015" H 5200 2600 50  0001 C CNN
 F 1 "+5V" V 5215 2878 50  0000 L CNN
 F 2 "" H 5200 2750 50  0001 C CNN
@@
 P 1650 1100
 AR Path="/5FDF6408/5FDC9F6E" Ref="#PWR?"  Part="1"
-AR Path="/5FDBBE2F/5FDC9F6E" Ref="#PWR0171"  Part="1"
-F 0 "#PWR0171" H 1650 950 50  0001 C CNN
+AR Path="/5FDBBE2F/5FDC9F6E" Ref="#PWR09"  Part="1"
+F 0 "#PWR09" H 1650 950 50  0001 C CNN
 F 1 "+5V" V 1665 1228 50  0000 L CNN
 F 2 "" H 1650 1100 50  0001 C CNN
@@
 P 1650 1500
 AR Path="/5ED37B53/5FB5AC07/5FDCAA12" Ref="#PWR?"  Part="1"
-AR Path="/5FDBBE2F/5FDCAA12" Ref="#PWR0172"  Part="1"
-F 0 "#PWR0172" H 1650 1250 50  0001 C CNN
+AR Path="/5FDBBE2F/5FDCAA12" Ref="#PWR010"  Part="1"
+F 0 "#PWR010" H 1650 1250 50  0001 C CNN
 F 1 "GND" V 1655 1372 50  0000 R CNN
 F 2 "" H 1650 1500 50  0001 C CNN
@@
 Connection ~ 1650 1500
 $Comp
-L Device:C C?
+L Device:C C10
 U 1 1 5FDCBA9F
 P 1350 1300
-F 0 "C?" H 1465 1346 50  0000 L CNN
+F 0 "C10" H 1465 1346 50  0000 L CNN
 F 1 "100n" H 1465 1255 50  0000 L CNN
-F 2 "" H 1388 1150 50  0001 C CNN
+F 2 "Capacitor_SMD:C_0603_1608Metric" H 1388 1150 50  0001 C CNN
 F 3 "~" H 1350 1300 50  0001 C CNN
 	1    1350 1300
@@
 	1350 1450 1350 1500
 $Comp
-L Device:C C?
+L Device:C C11
 U 1 1 5FDCC13F
 P 1950 1300
-F 0 "C?" H 2065 1346 50  0000 L CNN
+F 0 "C11" H 2065 1346 50  0000 L CNN
 F 1 "100n" H 2065 1255 50  0000 L CNN
-F 2 "" H 1988 1150 50  0001 C CNN
+F 2 "Capacitor_SMD:C_0603_1608Metric" H 1988 1150 50  0001 C CNN
 F 3 "~" H 1950 1300 50  0001 C CNN
 	1    1950 1300
@@
 	1950 1450 1950 1500
 $Comp
-L Device:R R?
+L Device:R R2
 U 1 1 5FDD01CA
 P 5800 2650
-F 0 "R?" V 5593 2650 50  0000 C CNN
+F 0 "R2" V 5593 2650 50  0000 C CNN
 F 1 "1k" V 5684 2650 50  0000 C CNN
-F 2 "" V 5730 2650 50  0001 C CNN
+F 2 "Resistor_SMD:R_0603_1608Metric" V 5730 2650 50  0001 C CNN
 F 3 "~" H 5800 2650 50  0001 C CNN
 	1    5800 2650
 	0    1    1    0
 $EndComp
-Wire Wire Line
-	5950 2650 6250 2650
-$Comp
-L thonkiconn_jackSocket_fuzzySi:fuzzySI_thonkiconn J?
-U 1 1 5FDD72CF
-P 6450 3700
-AR Path="/5ED37B53/5FB5AC07/5FDD72CF" Ref="J?"  Part="1"
-AR Path="/5FDBBE2F/5FDD72CF" Ref="J?"  Part="1"
-F 0 "J?" H 6162 3676 50  0000 R CNN
-F 1 "TRIGGER_OUT_B" H 6162 3767 50  0000 R CNN
-F 2 "" H 6700 3800 50  0001 C CNN
-F 3 "" H 6700 3800 50  0001 C CNN
-	1    6450 3700
-	-1   0    0    1
-$EndComp
-$Comp
-L power:GND #PWR?
-U 1 1 5FDD72D5
-P 6650 3500
-AR Path="/5ED37B53/5FB5AC07/5FDD72D5" Ref="#PWR?"  Part="1"
-AR Path="/5FDBBE2F/5FDD72D5" Ref="#PWR0173"  Part="1"
-F 0 "#PWR0173" H 6650 3250 50  0001 C CNN
-F 1 "GND" V 6655 3372 50  0000 R CNN
-F 2 "" H 6650 3500 50  0001 C CNN
-F 3 "" H 6650 3500 50  0001 C CNN
-	1    6650 3500
-	-1   0    0    1
-$EndComp
-Wire Wire Line
-	6650 3500 6650 3550
-Wire Wire Line
-	6250 3700 6250 3550
-Wire Wire Line
-	6250 3550 6650 3550
-Connection ~ 6650 3550
-Wire Wire Line
-	6650 3550 6650 3600
 Wire Wire Line
 	5200 3800 5650 3800
@@
 P 4200 3800
 AR Path="/5ED37B53/5FB5AC07/5FDD72E1" Ref="#PWR?"  Part="1"
-AR Path="/5FDBBE2F/5FDD72E1" Ref="#PWR0174"  Part="1"
-F 0 "#PWR0174" H 4200 3550 50  0001 C CNN
+AR Path="/5FDBBE2F/5FDD72E1" Ref="#PWR013"  Part="1"
+F 0 "#PWR013" H 4200 3550 50  0001 C CNN
 F 1 "GND" V 4205 3672 50  0000 R CNN
 F 2 "" H 4200 3800 50  0001 C CNN
@@
 $EndComp
 $Comp
-L SN74AHCT1G125DBVR:SN74AHCT1G125DBVR IC?
+L SN74AHCT1G125DBVR:SN74AHCT1G125DBVR IC2
 U 1 1 5FDD72EF
 P 4200 3800
-F 0 "IC?" H 4700 4065 50  0000 C CNN
+F 0 "IC2" H 4700 4065 50  0000 C CNN
 F 1 "SN74AHCT1G125DBVR" H 4700 3974 50  0000 C CNN
-F 2 "SOT95P280X145-5N" H 5050 3900 50  0001 L CNN
+F 2 "SN74AHCT1G125DBVR:SOT95P280X145-5N" H 5050 3900 50  0001 L CNN
 F 3 "http://www.ti.com/lit/ds/symlink/sn74ahct1g125.pdf" H 5050 3800 50  0001 L CNN
 F 4 "74AHCT Single Tri-state Bus Buffer SOT23 SN74AHCT1G125DBVR, Bus Buffer, HCT, 8.5 ns@ 50 pF, 8mA 4.5 ??? 5.5 V 5-Pin SOT-23" H 5050 3700 50  0001 L CNN "Description"
@@
 P 4200 4000
 AR Path="/5ED37B53/5FB5AC07/5FDD72F5" Ref="#PWR?"  Part="1"
-AR Path="/5FDBBE2F/5FDD72F5" Ref="#PWR0175"  Part="1"
-F 0 "#PWR0175" H 4200 3750 50  0001 C CNN
+AR Path="/5FDBBE2F/5FDD72F5" Ref="#PWR014"  Part="1"
+F 0 "#PWR014" H 4200 3750 50  0001 C CNN
 F 1 "GND" V 4205 3872 50  0000 R CNN
 F 2 "" H 4200 4000 50  0001 C CNN
@@
 P 5200 3900
 AR Path="/5FDF6408/5FDD72FB" Ref="#PWR?"  Part="1"
-AR Path="/5FDBBE2F/5FDD72FB" Ref="#PWR0176"  Part="1"
-F 0 "#PWR0176" H 5200 3750 50  0001 C CNN
+AR Path="/5FDBBE2F/5FDD72FB" Ref="#PWR016"  Part="1"
+F 0 "#PWR016" H 5200 3750 50  0001 C CNN
 F 1 "+5V" V 5215 4028 50  0000 L CNN
 F 2 "" H 5200 3900 50  0001 C CNN
@@
 	4200 3900 3850 3900
 $Comp
-L Device:R R?
+L Device:R R3
 U 1 1 5FDD7302
 P 5800 3800
-F 0 "R?" V 5593 3800 50  0000 C CNN
+F 0 "R3" V 5593 3800 50  0000 C CNN
 F 1 "1k" V 5684 3800 50  0000 C CNN
-F 2 "" V 5730 3800 50  0001 C CNN
+F 2 "Resistor_SMD:R_0603_1608Metric" V 5730 3800 50  0001 C CNN
 F 3 "~" H 5800 3800 50  0001 C CNN
 	1    5800 3800
 	0    1    1    0
 $EndComp
-Wire Wire Line
-	5950 3800 6250 3800
+$Comp
+L Connector:AudioJack2_SwitchT J?
+U 1 1 5FF01C3E
+P 6550 2650
+AR Path="/5ED4085B/5FF01C3E" Ref="J?"  Part="1"
+AR Path="/5ED37B53/5FB5AC07/5FF01C3E" Ref="J?"  Part="1"
+AR Path="/5FDBBE2F/5FF01C3E" Ref="J1"  Part="1"
+F 0 "J1" H 6370 2583 50  0000 R CNN
+F 1 "PJ398SM" H 6370 2674 50  0000 R CNN
+F 2 "Connector_Audio:Jack_3.5mm_QingPu_WQP-PJ398SM_Vertical_CircularHoles" H 6550 2650 50  0001 C CNN
+F 3 "~" H 6550 2650 50  0001 C CNN
+	1    6550 2650
+	-1   0    0    1
+$EndComp
+Wire Wire Line
+	5950 2650 6350 2650
+Wire Wire Line
+	6350 2750 6350 2800
+$Comp
+L power:GND #PWR?
+U 1 1 5FF01C46
+P 6350 2900
+AR Path="/5ED37B53/5FB5AC07/5FF01C46" Ref="#PWR?"  Part="1"
+AR Path="/5FDBBE2F/5FF01C46" Ref="#PWR017"  Part="1"
+F 0 "#PWR017" H 6350 2650 50  0001 C CNN
+F 1 "GND" V 6355 2772 50  0000 R CNN
+F 2 "" H 6350 2900 50  0001 C CNN
+F 3 "" H 6350 2900 50  0001 C CNN
+	1    6350 2900
+	1    0    0    -1
+$EndComp
+Wire Wire Line
+	6350 2550 6200 2550
+Wire Wire Line
+	6200 2550 6200 2800
+Wire Wire Line
+	6200 2800 6350 2800
+Connection ~ 6350 2800
+Wire Wire Line
+	6350 2800 6350 2900
+$Comp
+L Connector:AudioJack2_SwitchT J?
+U 1 1 5FF04587
+P 6550 3800
+AR Path="/5ED4085B/5FF04587" Ref="J?"  Part="1"
+AR Path="/5ED37B53/5FB5AC07/5FF04587" Ref="J?"  Part="1"
+AR Path="/5FDBBE2F/5FF04587" Ref="J2"  Part="1"
+F 0 "J2" H 6370 3733 50  0000 R CNN
+F 1 "PJ398SM" H 6370 3824 50  0000 R CNN
+F 2 "Connector_Audio:Jack_3.5mm_QingPu_WQP-PJ398SM_Vertical_CircularHoles" H 6550 3800 50  0001 C CNN
+F 3 "~" H 6550 3800 50  0001 C CNN
+	1    6550 3800
+	-1   0    0    1
+$EndComp
+Wire Wire Line
+	5950 3800 6350 3800
+Wire Wire Line
+	6350 3900 6350 3950
+$Comp
+L power:GND #PWR?
+U 1 1 5FF0458F
+P 6350 4050
+AR Path="/5ED37B53/5FB5AC07/5FF0458F" Ref="#PWR?"  Part="1"
+AR Path="/5FDBBE2F/5FF0458F" Ref="#PWR018"  Part="1"
+F 0 "#PWR018" H 6350 3800 50  0001 C CNN
+F 1 "GND" V 6355 3922 50  0000 R CNN
+F 2 "" H 6350 4050 50  0001 C CNN
+F 3 "" H 6350 4050 50  0001 C CNN
+	1    6350 4050
+	1    0    0    -1
+$EndComp
+Wire Wire Line
+	6350 3700 6200 3700
+Wire Wire Line
+	6200 3700 6200 3950
+Wire Wire Line
+	6200 3950 6350 3950
+Connection ~ 6350 3950
+Wire Wire Line
+	6350 3950 6350 4050
 $EndSCHEMATC

Commit message: Last adjustments to hardware before v0.1 release
Parts:
- C10, C11: LCSC (none) -> C14663; LCSC Part # (none) -> C14663
- R2, R3: LCSC (none) -> C21190; LCSC Part # (none) -> C21190
Changed lines of the file:
@@
 P 4200 2650
 AR Path="/5ED37B53/5FB5AC07/5FDC3D71" Ref="#PWR?"  Part="1"
-AR Path="/5FDBBE2F/5FDC3D71" Ref="#PWR011"  Part="1"
-F 0 "#PWR011" H 4200 2400 50  0001 C CNN
+AR Path="/5FDBBE2F/5FDC3D71" Ref="#PWR015"  Part="1"
+F 0 "#PWR015" H 4200 2400 50  0001 C CNN
 F 1 "GND" V 4205 2522 50  0000 R CNN
 F 2 "" H 4200 2650 50  0001 C CNN
@@
 P 4200 2850
 AR Path="/5ED37B53/5FB5AC07/5FDC7341" Ref="#PWR?"  Part="1"
-AR Path="/5FDBBE2F/5FDC7341" Ref="#PWR012"  Part="1"
-F 0 "#PWR012" H 4200 2600 50  0001 C CNN
+AR Path="/5FDBBE2F/5FDC7341" Ref="#PWR016"  Part="1"
+F 0 "#PWR016" H 4200 2600 50  0001 C CNN
 F 1 "GND" V 4205 2722 50  0000 R CNN
 F 2 "" H 4200 2850 50  0001 C CNN
@@
 P 5200 2750
 AR Path="/5FDF6408/5FDC8A1E" Ref="#PWR?"  Part="1"
-AR Path="/5FDBBE2F/5FDC8A1E" Ref="#PWR015"  Part="1"
-F 0 "#PWR015" H 5200 2600 50  0001 C CNN
+AR Path="/5FDBBE2F/5FDC8A1E" Ref="#PWR019"  Part="1"
+F 0 "#PWR019" H 5200 2600 50  0001 C CNN
 F 1 "+5V" V 5215 2878 50  0000 L CNN
 F 2 "" H 5200 2750 50  0001 C CNN
@@
 P 1650 1100
 AR Path="/5FDF6408/5FDC9F6E" Ref="#PWR?"  Part="1"
-AR Path="/5FDBBE2F/5FDC9F6E" Ref="#PWR09"  Part="1"
-F 0 "#PWR09" H 1650 950 50  0001 C CNN
+AR Path="/5FDBBE2F/5FDC9F6E" Ref="#PWR013"  Part="1"
+F 0 "#PWR013" H 1650 950 50  0001 C CNN
 F 1 "+5V" V 1665 1228 50  0000 L CNN
 F 2 "" H 1650 1100 50  0001 C CNN
@@
 P 1650 1500
 AR Path="/5ED37B53/5FB5AC07/5FDCAA12" Ref="#PWR?"  Part="1"
-AR Path="/5FDBBE2F/5FDCAA12" Ref="#PWR010"  Part="1"
-F 0 "#PWR010" H 1650 1250 50  0001 C CNN
+AR Path="/5FDBBE2F/5FDCAA12" Ref="#PWR014"  Part="1"
+F 0 "#PWR014" H 1650 1250 50  0001 C CNN
 F 1 "GND" V 1655 1372 50  0000 R CNN
 F 2 "" H 1650 1500 50  0001 C CNN
@@
 F 2 "Capacitor_SMD:C_0603_1608Metric" H 1388 1150 50  0001 C CNN
 F 3 "~" H 1350 1300 50  0001 C CNN
+F 4 "C14663" H 1350 1300 50  0001 C CNN "LCSC Part #"
+F 5 "C14663" H 1350 1300 50  0001 C CNN "LCSC"
 	1    1350 1300
 	1    0    0    -1
@@
 F 2 "Capacitor_SMD:C_0603_1608Metric" H 1988 1150 50  0001 C CNN
 F 3 "~" H 1950 1300 50  0001 C CNN
+F 4 "C14663" H 1950 1300 50  0001 C CNN "LCSC Part #"
+F 5 "C14663" H 1950 1300 50  0001 C CNN "LCSC"
 	1    1950 1300
 	1    0    0    -1
@@
 F 2 "Resistor_SMD:R_0603_1608Metric" V 5730 2650 50  0001 C CNN
 F 3 "~" H 5800 2650 50  0001 C CNN
+F 4 "C21190" H 5800 2650 50  0001 C CNN "LCSC Part #"
+F 5 "C21190" H 5800 2650 50  0001 C CNN "LCSC"
 	1    5800 2650
 	0    1    1    0
@@
 P 4200 3800
 AR Path="/5ED37B53/5FB5AC07/5FDD72E1" Ref="#PWR?"  Part="1"
-AR Path="/5FDBBE2F/5FDD72E1" Ref="#PWR013"  Part="1"
-F 0 "#PWR013" H 4200 3550 50  0001 C CNN
+AR Path="/5FDBBE2F/5FDD72E1" Ref="#PWR017"  Part="1"
+F 0 "#PWR017" H 4200 3550 50  0001 C CNN
 F 1 "GND" V 4205 3672 50  0000 R CNN
 F 2 "" H 4200 3800 50  0001 C CNN
@@
 P 4200 4000
 AR Path="/5ED37B53/5FB5AC07/5FDD72F5" Ref="#PWR?"  Part="1"
-AR Path="/5FDBBE2F/5FDD72F5" Ref="#PWR014"  Part="1"
-F 0 "#PWR014" H 4200 3750 50  0001 C CNN
+AR Path="/5FDBBE2F/5FDD72F5" Ref="#PWR018"  Part="1"
+F 0 "#PWR018" H 4200 3750 50  0001 C CNN
 F 1 "GND" V 4205 3872 50  0000 R CNN
 F 2 "" H 4200 4000 50  0001 C CNN
@@
 P 5200 3900
 AR Path="/5FDF6408/5FDD72FB" Ref="#PWR?"  Part="1"
-AR Path="/5FDBBE2F/5FDD72FB" Ref="#PWR016"  Part="1"
-F 0 "#PWR016" H 5200 3750 50  0001 C CNN
+AR Path="/5FDBBE2F/5FDD72FB" Ref="#PWR020"  Part="1"
+F 0 "#PWR020" H 5200 3750 50  0001 C CNN
 F 1 "+5V" V 5215 4028 50  0000 L CNN
 F 2 "" H 5200 3900 50  0001 C CNN
@@
 F 2 "Resistor_SMD:R_0603_1608Metric" V 5730 3800 50  0001 C CNN
 F 3 "~" H 5800 3800 50  0001 C CNN
+F 4 "C21190" H 5800 3800 50  0001 C CNN "LCSC Part #"
+F 5 "C21190" H 5800 3800 50  0001 C CNN "LCSC"
 	1    5800 3800
 	0    1    1    0
@@
 P 6350 2900
 AR Path="/5ED37B53/5FB5AC07/5FF01C46" Ref="#PWR?"  Part="1"
-AR Path="/5FDBBE2F/5FF01C46" Ref="#PWR017"  Part="1"
-F 0 "#PWR017" H 6350 2650 50  0001 C CNN
+AR Path="/5FDBBE2F/5FF01C46" Ref="#PWR021"  Part="1"
+F 0 "#PWR021" H 6350 2650 50  0001 C CNN
 F 1 "GND" V 6355 2772 50  0000 R CNN
 F 2 "" H 6350 2900 50  0001 C CNN
@@
 P 6350 4050
 AR Path="/5ED37B53/5FB5AC07/5FF0458F" Ref="#PWR?"  Part="1"
-AR Path="/5FDBBE2F/5FF0458F" Ref="#PWR018"  Part="1"
-F 0 "#PWR018" H 6350 3800 50  0001 C CNN
+AR Path="/5FDBBE2F/5FF0458F" Ref="#PWR022"  Part="1"
+F 0 "#PWR022" H 6350 3800 50  0001 C CNN
 F 1 "GND" V 6355 3922 50  0000 R CNN
 F 2 "" H 6350 4050 50  0001 C CNN
